File: v1.backup.sch$9.sch (EAGLE design)
At the start: 245 parts, among them J1 DC-044-A, J2 MICROSD-9P, J3 2p-2.54, J4 2p-2.54, J5 16p-2.54, J6 16p-2.54, J7 2x3p-2.54, J8 2p-2.54, Q2 SSM3J328R,LF, Q3 6pF@32.7680kHz, Q4 BSS138W-7-F, Q5 SSM3J328R,LF, SW1 SW-200D, SW2 SW-200D, SW3 SW-200D, SW4 SW-200D, SW5 SW-200D, SW6 SW-200D, SW7 SW-200D, SW8 SW-200D, U1 MCP23017-E/SO, U10 74HC139N, U11 BZX84C30, U12 SP483ECN-L, U13 FT232RL-SSOP28, U14 FT232RL-SSOP28, U15 FT232RL-SSOP28, U2 MCP79412-I/SN, U3 LOPY, U5 FT232RL-SSOP28, U6 FT232RL-SSOP28, U7 2x14p-2.54, U8 BR24G32-3, X1 JST-XH-05-PIN-ROUND-PAD, X10 JST-XH-07-PIN-ROUND-PAD, X11 JST-XH-07-PIN-ROUND-PAD, X12 JST-XH-07-PIN-ROUND-PAD, X13 JST-XH-05-PIN-ROUND-PAD, X14 JST-XH-05-PIN-ROUND-PAD, X15 JST-XH-05-PIN-ROUND-PAD, X16 JST-XH-05-PIN-ROUND-PAD, X17 JST-XH-05-PIN-ROUND-PAD, X18 JST-XH-05-PIN-ROUND-PAD, X19 JST-XH-05-PIN-ROUND-PAD, X2 JST-XH-05-PIN-ROUND-PAD, X20 JST-XH-05-PIN-ROUND-PAD, X21 JST-XH-05-PIN-ROUND-PAD, X22 JST-XH-07-PIN-ROUND-PAD, X23 JST-XH-05-PIN-ROUND-PAD, X24 JST-XH-07-PIN-ROUND-PAD, X25 JST-XH-07-PIN-ROUND-PAD, X26 JST-XH-05-PIN-ROUND-PAD, X27 JST-XH-07-PIN-ROUND-PAD, X28 JST-XH-05-PIN-ROUND-PAD, X29 JST-XH-05-PIN-ROUND-PAD, X3 JST-XH-05-PIN-ROUND-PAD, X30 JST-XH-05-PIN-ROUND-PAD, X31 JST-XH-05-PIN-ROUND-PAD, X4 JST-XH-07-PIN-ROUND-PAD, X5 JST-XH-07-PIN-ROUND-PAD, X6 JST-XH-07-PIN-ROUND-PAD, X7 JST-XH-07-PIN-ROUND-PAD, X8 JST-XH-07-PIN-ROUND-PAD, X9 JST-XH-07-PIN-ROUND-PAD, Y2 12MHZ

Commit message: starting board layout
Connections:
- removed net N$124: F17.2, X19-1.S
- removed net N$126: F19.2, X20-1.S
- removed net N$17: F21.2, X21-1.S
- removed net N$48 (its old number): F5.2, X13-1.S
- removed net N$50 (its old number): F7.2, X14-1.S
- removed net N$52 (its old number): F9.2, X15-1.S
- removed net N$54 (its old number): F11.2, X16-1.S
- removed net N$78: F13.2, X17-1.S
- new net N$120: R38.1, U8.SDA
- new net N$127: Q4.S
- new net N$89: SW3.1
- net +3V3_SMOOTH: now also R10.2
- net +5V: now also F11.2, F13.2, F15.2, F17.2, F19.2, F21.2, F36.2, F5.2, F7.2, F9.2, X13-1.S, X14-1.S, X15-1.S, X16-1.S, X17-1.S, X18-1.S, X19-1.S, X20-1.S, X21-1.S, X23-1.S
- net 3V3_SMOOTH: no longer R10.2
- net GND: no longer Q4.S, R40.1
- net ID_SC: no longer R37.1, U8.SCL
- net ID_SD: no longer R38.1, U8.SDA
- net N$119: now also R37.1, U8.SCL; no longer F15.2, X18-1.S
- net N$128: now also R40.1; no longer F36.2, X23-1.S
- net N$86: no longer SW3.1
Other:
- moved on the sheet: F10, F11, F12, F13, F14, F15, F16, F17, F18, F19, F20, F36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
