File: v2.0.brd (EAGLE design)
At the start: 245 x 105 mm, 289 parts, among them J1 DC-044-A, J10 16p-2.54, J11 16p-2.54, J2 MICROSD-9P, J3 2p-2.54, J4 2p-2.54, J5 16p-2.54, J6 16p-2.54, J7 16p-2.54, J8 2p-2.54, J9 16p-2.54, Q1 32.768khZ@6Pf, Q10 S8550, Q2 SSM3J328R,LF, Q3 BSS138W-7-F, Q4 BSS138W-7-F, Q5 SSM3J328R,LF, Q6 BSS138W-7-F, Q7 BSS138W-7-F, Q8 CJ2305, Q9 S8550, SW1 MK-12C02 G1.5, SW2 MK-12C02 G1.5, SW3 MK-12C02 G1.5, SW4 MK-12C02 G1.5, U1 MCP23017-E/SO, U10 74HCT139D, U11 BZX84C30, U12 SP483ECN-L, U13 FT232RL-SSOP28, U14 FT232RL-SSOP28, U15 FT232RL-SSOP28, U2 MCP79412-I/SN, U3 LOPY, U4 MAX213IDBR, U5 FT232RL-SSOP28, U6 FT232RL-SSOP28, U8 BR24G32-3, Y2 12MHZ

Commit message: Start of connector / fuse rationalisation
Parts:
- removed C15, C16: 100nf, Seeed-Capacitor-2016:C0603
- removed C17: 4.7uf, Seeed-Capacitor:AVX-A
- removed C9: 10nf, Seeed-Capacitor-2016:C0805
- removed D10: RED-0603, Seeed-LED-2016:LED-0603
- removed D2: BLUE-0603, Seeed-LED:LED-0603
- removed D3: GREEN-0603, Seeed-LED:LED-0603
- removed F11, F12, F13, F14, F17, F18, F2, F21, F22, F23, F24, F25, F3, F30, F31, F32, F33, F34, F35, F36, F37, F38, F39, F4, F44, F45, F52, F53, F7, F8, F80, F81: SMD1206R500SF, Seeed-Fuse:F1206
- removed I2C_10, I2C_5: JST-XH-05-PIN-ROUND-PAD, Rembrandt Electronics - JST XH Connectors v1-0 2:JST-XH-05-PACKAGE-ROUND-PAD
- removed L1: 330R-1500MA, Seeed-Inductor-2016:L0805
- removed R1, R3: 330R, Seeed-Resistor:R0603
- removed R11: 1K, Seeed-Resistor-2016:R0603
- removed R13, R14: 0R, Seeed-Resistor:R0603
- removed SPI_3, SPI_4, SPI_7, SPI_8: JST-XH-07-PIN-ROUND-PAD, Rembrandt Electronics - JST XH Connectors v1-0 2:JST-XH-07-PACKAGE-ROUND-PAD
- removed TP5: TPB2,54, testpad:B2,54
- removed U6: FT232RL-SSOP28, Seeed-IC:SSOP28-0.65-10.2X5.2MM
- removed USB3: ZX62-B-5PA, Seeed-Connector -2016:MICRO-USB5+6P-SMD-0.65-AB
- added J12: 4p-2.54, Seeed-Connector:H4-2.54
- added JP1: (no value), jumper:JP1
- moved SPI_1 50.0 mm to (43.7, 87.1)
- moved SPI_2 47.0 mm to (51.6, 87.1)
- moved TP3 44.7 mm to (98.3, 91.9)
- moved F29 40.6 mm to (38.6, 90.8)
- moved F28 40.5 mm to (38.5, 96.1)
- moved U10 32.5 mm to (70.9, 70.4)
- moved SPI_5 24.9 mm to (63.0, 87.1)
- moved F26 24.6 mm to (57.7, 96.1)
- moved F27 24.6 mm to (57.7, 90.8)
- moved F41 24.5 mm to (99.8, 69.0), turned to 90 degrees
- moved SPI_6 22.4 mm to (71.6, 87.1)
- moved C13 20.6 mm to (65.0, 73.8), turned to 0 degrees
- moved TP12 5.59 mm to (109.0, 97.0)
- moved F43 1.97 mm to (95.6, 68.8)
- moved F42 1.59 mm to (89.5, 67.6), turned to 180 degrees
Connections:
- removed net ADC_2_3V3_P: F39.2, PI_ADC_2.2
- removed net ADC_2_5V_P: F38.2, PI_ADC_2.1
- removed net ADC_3_3V3_P: F43.2, PI_ADC_3.2
- removed net ADC_4_5V_P: F44.2, PI_ADC_4.1
- removed net FTDI1_3V3: C16.2, U6.17
- removed net LOPY_UART1_3V3_PROTECTED: F81.2, LOPY_UART1.2
- removed net LOPY_UART1_5V_PROTECTED: F80.2, LOPY_UART1.1
- removed net LOPY_USB_5V: C15.2, C17.+, L1.2, R1.1, R11.2, R3.1, TP5.TP, U6.20, U6.4
- removed net N$10: R14.1, U6.5
- removed net N$2: D3.-, U6.22
- removed net N$3: D2.-, U6.23
- removed net N$6: D3.+, R3.2
- removed net N$7: D2.+, R1.2
- removed net N$77: D10.+, R11.1
- removed net N$8: R13.1, U6.1
- removed net PI_I2C_3V3_1: F8.2, I2C_2.2
- removed net PI_I2C_3V3_10: F37.2, I2C_10.2
- removed net PI_I2C_3V3_4: F12.2, I2C_4.2
- removed net PI_I2C_3V3_5: F14.2, I2C_5.2
- removed net PI_I2C_3V3_7: F18.2, I2C_7.2
- removed net PI_I2C_3V3_9: F22.2, I2C_9.2
- removed net PI_I2C_5V_P1: F7.2, I2C_2.1
- removed net PI_I2C_5V_P3: F11.2, I2C_4.1
- removed net PI_I2C_5V_P4: F13.2, I2C_5.1
- removed net PI_I2C_5V_P6: F17.2, I2C_7.1
- removed net PI_I2C_5V_P8: F21.2, I2C_9.1
- removed net PI_I2C_5V_P9: F36.2, I2C_10.1
- removed net PI_SPI_5V_2_P: F2.2, SPI_2.1
- removed net PI_UART_HUB_2_3V3_P: F53.2, PI_UART_HUB_2.2
- removed net PI_UART_HUB_2_5V_P: F52.2, PI_UART_HUB_2.1
- removed net RPI_CS8: SPI_8.3, U10.9
- removed net SPI_3V3_2_P: F3.2, SPI_2.2
- removed net SPI_3V3_3_P: F23.2, SPI_3.2
- removed net SPI_3V3_4_P: F25.2, SPI_4.2
- removed net SPI_3V3_6_P: F31.2, SPI_6.2
- removed net SPI_3V3_7_P: F33.2, SPI_7.2
- removed net SPI_3V3_8_P: F35.2, SPI_8.2
- removed net SPI_5V_3_P: F4.2, SPI_3.1
- removed net SPI_5V_4_P: F24.2, SPI_4.1
- removed net SPI_5V_6_P: F30.2, SPI_6.1
- removed net SPI_5V_7_P: F32.2, SPI_7.1
- removed net SPI_5V_8_P: F34.2, SPI_8.1
- removed net USB_DM: U6.16, USB3.2
- removed net USB_DP: U6.15, USB3.3
- removed net VBUS: C9.2, L1.1, USB3.1
- new net RPI_CS0: SPI_1.3, U10.4
- net +3V3: no longer F12.1, F14.1, F18.1, F22.1, F23.1, F25.1, F3.1, F31.1, F33.1, F35.1, F37.1, F53.1, F8.1
- net +3V3_SMOOTH: no longer F39.1, F45.1
- net +5V: now also JP1.1; no longer F80.1
- net ADC_1_3V3_P: now also PI_ADC_2.2
- net ADC_1_5V_P: now also PI_ADC_2.1
- net ADC_3_5V_P: now also PI_ADC_4.1
- net ADC_4_3V3_P: now also F43.2, PI_ADC_3.2; no longer F45.2
- net GND: now also JP1.2; no longer C15.1, C16.1, C17.-, C9.1, I2C_10.5, I2C_5.5, SPI_3.7, SPI_4.7, SPI_7.7, SPI_8.7, U6.18, U6.21, U6.25, U6.26, U6.7, USB3.5, USB3.P1, USB3.P2, USB3.P3, USB3.P4, USB3.P5, USB3.P6
- net LED_GND: no longer D10.-
- net LOPY_3V3: no longer F81.1
- net LOPY_RXD0: no longer R13.2
- net LOPY_TXD0: no longer R14.2
- net LOPY_UART0_3V3_PROTECTED: now also LOPY_UART1.2
- net LOPY_UART0_5V_PROTECTED: now also LOPY_UART1.1
- net PI_5V: no longer F11.1, F13.1, F17.1, F2.1, F21.1, F24.1, F30.1, F32.1, F34.1, F36.1, F38.1, F4.1, F44.1, F52.1, F7.1
- net PI_5V_SPI_1_P: now also SPI_2.1
- net PI_I2C_3V3_2: now also I2C_4.2
- net PI_I2C_3V3_3: now also I2C_2.2
- net PI_I2C_3V3_6: now also I2C_7.2
- net PI_I2C_3V3_8: now also I2C_9.2
- net PI_I2C_5V_P: now also I2C_2.1
- net PI_I2C_5V_P2: now also I2C_4.1
- net PI_I2C_5V_P5: now also I2C_7.1
- net PI_I2C_5V_P7: now also I2C_9.1
- net PI_SPI_3V3_1_P: now also SPI_2.2
- net PI_UART_HUB_1_3V3_P: now also PI_UART_HUB_2.2
- net PI_UART_HUB_1_5V_P: now also PI_UART_HUB_2.1
- net RPI_CS1: now also SPI_2.3, U10.5; no longer SPI_1.3, U10.4
- net RPI_CS2: now also SPI_5.3, U10.6; no longer SPI_2.3, U10.5
- net RPI_CS3: now also SPI_6.3, U10.7; no longer SPI_3.3, U10.6
- net RPI_CS4: now also J12.1, U10.12; no longer SPI_4.3, U10.7
- net RPI_CS5: now also J12.2, U10.11; no longer SPI_5.3, U10.12
- net RPI_CS6: now also J12.3, U10.10; no longer SPI_6.3, U10.11
- net RPI_CS7: now also J12.4, U10.9; no longer SPI_7.3, U10.10
- net SCL_3V3: no longer I2C_10.4, I2C_5.4
- net SDA_3V3: no longer I2C_10.3, I2C_5.3
- net SPI_3V3_5_P: now also SPI_6.2
- net SPI_5V_5_P: now also SPI_6.1
- net SPI_MISO: no longer SPI_3.5, SPI_4.5, SPI_7.5, SPI_8.5
- net SPI_MOSI: no longer SPI_3.4, SPI_4.4, SPI_7.4, SPI_8.4
- net SPI_SCLK: no longer SPI_3.6, SPI_4.6, SPI_7.6, SPI_8.6
Routing:
- net LED_GND: track 584.4 -> 337.0 mm, vias 11 -> 6
- net PI_5V: track 536.8 -> 413.2 mm, vias 9 -> 7
- net +3V3: track 678.9 -> 578.8 mm, vias 27 -> 23
- net SPI_MOSI: track 205.4 -> 147.0 mm
- net LOPY_USB_5V: track 54.1 -> 0.00 mm
- net SPI_SCLK: track 208.1 -> 158.0 mm
- net SPI_MISO: track 204.5 -> 154.4 mm
- net SCL_3V3: track 287.2 -> 241.9 mm, vias 5 -> 4
- net GND: track 43.7 -> 0.00 mm, vias 51 -> 27
- net RPI_CS0: track 0.00 -> 43.3 mm
- net RPI_CS8: track 43.1 -> 0.00 mm
- net SDA_3V3: track 259.8 -> 220.9 mm, vias 4 -> 5
- net SPI_GPIO4: track 174.4 -> 141.9 mm
- net SPI_GPIO3: track 174.0 -> 141.5 mm
- net SPI_GPIO2: track 179.4 -> 146.8 mm
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Other:
- board text added: "Spare CS"
- board text removed: "SPI4"
- board text removed: "SPI5"
- board text removed: "SPI6"
- board text removed: "SPI7"
- board text removed: "USB"
