File: v2.0.brd (EAGLE design)
At the start: 245 x 105 mm, 237 parts, among them J1 DC-044-A, J10 16p-2.54, J11 16p-2.54, J12 4p-2.54, J2 MICROSD-9P, J3 2p-2.54, J4 2p-2.54, J5 16p-2.54, J6 16p-2.54, J7 16p-2.54, J8 2p-2.54, J9 16p-2.54, Q1 32.768khZ@6Pf, Q10 S8550, Q2 SSM3J328R,LF, Q3 BSS138W-7-F, Q4 BSS138W-7-F, Q5 SSM3J328R,LF, Q6 BSS138W-7-F, Q7 BSS138W-7-F, Q8 CJ2305, Q9 S8550, SW1 MK-12C02 G1.5, SW2 MK-12C02 G1.5, SW3 MK-12C02 G1.5, SW4 MK-12C02 G1.5, U1 MCP23017-E/SO, U10 74HCT139D, U11 BZX84C30, U12 SP483ECN-L, U13 FT232RL-SSOP28, U14 FT232RL-SSOP28, U15 FT232RL-SSOP28, U2 MCP79412-I/SN, U3 LOPY, U4 MAX213IDBR, U5 FT232RL-SSOP28, U8 BR24G32-3, Y2 12MHZ

Commit message: More rearranging
Parts:
- removed J8: 2p-2.54, Seeed-Connector -2016:H2-2.54
- added F2: SMD1206R500SF, Seeed-Fuse:F1206
- moved JP1 178.9 mm to (89.2, 103.1), turned to 270 degrees
- moved TP2 80.7 mm to (77.5, 40.6)
- moved PI_UART 17.9 mm to (63.0, 16.3)
- moved F50 16.9 mm to (57.4, 22.9)
- moved F51 16.8 mm to (57.4, 17.5)
- moved PI_UART_HUB_2 14.0 mm to (51.6, 16.3)
- moved F55 12.8 mm to (80.5, 26.0), turned to 270 degrees
- moved F6 12.2 mm to (38.6, 56.0)
- moved I2C_1 12.2 mm to (43.7, 54.9)
- moved I2C_6 12.2 mm to (43.7, 35.3)
- moved F15 12.1 mm to (38.5, 41.8)
- moved F5 12.1 mm to (38.5, 61.3)
- moved F48 12.1 mm to (38.5, 22.9)
- moved F16 11.9 mm to (38.4, 36.3)
- moved F49 11.9 mm to (38.5, 17.4)
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Connections:
- new net N$2: F2.2, JP1.1
- net +5V: now also F2.1; no longer JP1.1
- net EEPROM_WP: no longer J8.1
- net GND: no longer J8.2
Routing:
- net +3V3: track 578.8 -> 462.8 mm, vias 23 -> 15
- net PI_5V: track 413.2 -> 494.2 mm, vias 7 -> 10
- net RXD2: track 78.9 -> 0.00 mm, vias 1 -> 0
- net TXD2: track 78.5 -> 0.00 mm, vias 1 -> 0
- net RXD1: track 78.1 -> 0.00 mm, vias 1 -> 0
- net TXD1: track 74.6 -> 0.00 mm, vias 1 -> 0
- net RS232_3_RXD: track 68.1 -> 0.00 mm, vias 1 -> 0
- net RS232_3_TXD: track 63.6 -> 0.00 mm, vias 1 -> 0
- net FTDI_HUB_LEDS: track 60.5 -> 26.2 mm, vias 2 -> 0
- net SDA_3V3: track 220.9 -> 230.5 mm, vias 5 -> 4
- net SCL_3V3: track 241.9 -> 232.6 mm, vias 4 -> 3
- net PI_I2C_5V_P2: track 5.13 -> 14.1 mm
- net PI_I2C_3V3_2: track 5.13 -> 14.1 mm
- net UART_HUB_3_3V3_P: track 5.01 -> 13.3 mm
- net PI_UART_HUB_1_5V_P: track 4.79 -> 13.1 mm
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
Commit message: V2 laid out
Parts:
- removed F74, F75: SMD1206R500SF, Seeed-Fuse:F1206
- moved D11 92.8 mm to (92.6, 6.99)
- moved R35 92.8 mm to (92.6, 5.21)
- moved C22 75.4 mm to (87.2, 14.5), turned to 180 degrees
- moved TP2 75.3 mm to (31.2, 100.1)
- moved C24 73.0 mm to (87.2, 10.8), turned to 0 degrees
- moved USB1 72.5 mm to (65.4, 1.47)
- moved L4 68.1 mm to (67.7, 6.48)
- moved C25 68.0 mm to (67.6, 8.51)
- moved C43 66.2 mm to (58.5, 4.95), turned to 270 degrees
- moved C44 64.2 mm to (61.1, 7.87)
- moved C42 62.7 mm to (58.0, 7.62), turned to 0 degrees
- moved C47 62.3 mm to (70.0, 10.9), turned to 180 degrees
- moved U4 61.2 mm to (80.0, 15.1), turned to 0 degrees
- moved C23 59.7 mm to (80.5, 8.38), turned to 270 degrees
- moved F76 53.6 mm to (29.3, 72.5), turned to 270 degrees
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Connections:
- net N$16 renamed P2_EN
- net N$18 renamed PI12_EN
- removed net LOPY_SPI_3V3_PROTECTED: F75.2, LOPY_SPI.2
- removed net LOPY_SPI_5V_PROTECTED: F74.2, LOPY_SPI.1
- net +5V: no longer F74.1
- net LOPY_3V3: no longer F75.1
- net LOPY_I2C_3V3_PROTECTED: now also LOPY_SPI.2
- net N$4: now also LOPY_SPI.1
- net N$9: now also SW1.A; no longer SW1.B
Routing:
- net LED_GND: track 337.0 -> 460.2 mm, vias 6 -> 9
- net RS232_3_LED1: track 103.8 -> 4.31 mm, vias 2 -> 0
- net RS232_3_LED2: track 105.0 -> 7.09 mm, vias 2 -> 0
- net RS232_2_LED2: track 98.9 -> 10.0 mm, vias 2 -> 0
- net RS232_2_LED1: track 94.0 -> 8.96 mm, vias 2 -> 0
- net LOPY_3V3: track 196.2 -> 125.7 mm, vias 10 -> 3
- net +5V: track 516.9 -> 458.8 mm
- net FTDI_HUB_LEDS: track 26.2 -> 80.4 mm, vias 0 -> 4
- net RS232_1_LED1: track 74.3 -> 28.8 mm
- net RS232_1_LED2: track 75.1 -> 32.7 mm
- net FTDI2_TXD: track 42.2 -> 2.34 mm, vias 2 -> 0
- net PI_TTL_RXD: track 222.5 -> 182.7 mm, vias 4 -> 1
- net SPI_GPIO4: track 141.9 -> 179.8 mm
- net PI_TTL_TXD: track 212.6 -> 174.8 mm, vias 4 -> 3
- net SPI_GPIO3: track 141.5 -> 174.8 mm
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Other:
- board size 245 x 105 mm -> 225 x 105 mm
- board text added: "Hub"

Commit message: RTC changed to one that doesn't rely on external crystal
Parts:
- removed C1, C3: 10pf, Seeed-Capacitor:C0603
- removed Q1: 32.768khZ@6Pf, imported-parts:85SMX
- added JP2: (no value), jumper:JP1
- U2: value MCP79412-I/SN -> DS3231SN; device imported-parts:SOIC127P600X175-8N -> imported-parts:SOIC127P1032X265-16N
- moved U2 7.41 mm to (105.4, 29.0), turned to 0 degrees
- moved C2 1.93 mm to (100.6, 37.1), turned to 0 degrees
- moved J2 1.27 mm to (0.28, 15.2)
Connections:
- removed net X1_RTC: C1.1, Q1.1, U2.1
- removed net X2_RTC: C3.1, Q1.4, U2.2
- net +3V3: now also U2.2; no longer U2.8
- net GND: now also JP2.1, JP2.2, U2.10, U2.11, U2.12, U2.13, U2.5, U2.6, U2.7, U2.8, U2.9; no longer C1.2, C3.2, U2.4
- net RTC_BATT: now also U2.14; no longer U2.3
- net SCL_3V3: now also U2.16; no longer U2.6
- net SDA_3V3: now also U2.15; no longer U2.5
Routing:
- net +3V3: track 491.9 -> 477.8 mm
- net X1_RTC: track 6.79 -> 0.00 mm
- net X2_RTC: track 6.59 -> 0.00 mm
- net RTC_BATT: track 60.2 -> 54.6 mm
- net P2_EN: track 353.8 -> 349.7 mm
- net SDA_3V3: track 221.8 -> 224.3 mm
- net SCL_3V3: track 231.3 -> 233.1 mm, vias 3 -> 5
- net LOPY_RXD1: track 90.2 -> 89.0 mm
- net LOPY_USD_SCLK: track 45.1 -> 43.9 mm
- net LOPY_CS1: track 33.6 -> 32.3 mm
- net LOPY_3V3: track 125.7 -> 124.5 mm
Other:
- board text added: "Pi-SEB"
- board text added: "USB LED"
- board text removed: "LED"

Commit message: More layout changes
Parts:
- moved F42 1.27 mm to (89.5, 68.8)
- moved C23 0.72 mm to (80.0, 8.89)
- moved D12 0.64 mm to (37.3, 15.2)
- moved TP17 0.51 mm to (96.2, 2.41)
- moved R42 0.25 mm to (37.3, 18.7)
- moved F28 0.13 mm to (38.6, 96.1)
Routing:
- net +3V3: track 477.8 -> 499.9 mm
- net GPIO4: track 78.8 -> 75.9 mm
- net ADC_3_5V_P: track 21.4 -> 22.6 mm
- net RS485_CBUS2: track 22.9 -> 24.1 mm
- net PI_5V: track 476.3 -> 475.1 mm
- net N$49: track 2.79 -> 1.91 mm
- net LED_GND: track 460.2 -> 459.5 mm
- net 5V_USB_HUB_FERRITE: track 190.1 -> 189.4 mm
- net RTC_BATT: track 54.6 -> 55.1 mm
Other:
- board text added: "05"
- board text added: "06"

Commit message: More layout tweaking
Parts:
- added PI_UART_HUB_1: JST-XH-05-PIN-ROUND-PAD, Rembrandt Electronics - JST XH Connectors v1-0 2:JST-XH-05-PACKAGE-ROUND-PAD
- added R1, R3: 0R, Seeed-Resistor:R0603
- added R11, R13: DNP, rcl:R0603
- moved PI_UART 50.3 mm to (30.2, 66.3)
- moved F51 35.8 mm to (30.6, 53.2), turned to 180 degrees
- moved F50 30.3 mm to (30.6, 49.1), turned to 180 degrees
- moved F76 16.1 mm to (13.3, 71.2)
Connections:
- new net RXD3_CONV: R13.1, U4.26
- new net TTL3_OUT_RXD: PI_UART_HUB_1.4, R3.2
- new net TTL3_OUT_TXD: PI_UART_HUB_1.3, R1.2
- new net TXD3_CONV: R11.1, U4.20
- net GND: now also PI_UART_HUB_1.5
- net RXD3: now also R13.2, R3.1; no longer U4.26
- net TXD3: now also R1.1, R11.2; no longer U4.20
- net UART_HUB_3_3V3_P: now also PI_UART_HUB_1.2
- net UART_USB_HUB_3_5V: now also PI_UART_HUB_1.1
Routing:
- net TTL3_OUT_TXD: track 0.00 -> 20.5 mm
- net TTL3_OUT_RXD: track 0.00 -> 20.4 mm, vias 0 -> 1
- net PI_UART_5V_P: track 5.72 -> 25.1 mm
- net TXD3: track 27.2 -> 41.8 mm
- net TXD3_CONV: track 0.00 -> 12.8 mm
- net PI_5V: track 475.1 -> 487.6 mm, vias 8 -> 10
- net FTDI_HUB_LEDS: track 80.4 -> 67.9 mm
- net PI_UART_3V3_P: track 5.72 -> 16.9 mm
- net PI_TTL_RXD: track 182.7 -> 173.2 mm, vias 1 -> 2
- net UART_USB_HUB_3_5V: track 10.7 -> 19.3 mm
- net UART_HUB_3_3V3_P: track 10.8 -> 19.4 mm
- net PI_TTL_TXD: track 174.8 -> 167.0 mm, vias 3 -> 1
- net RXD3_CONV: track 0.00 -> 6.29 mm
- net +3V3: track 499.9 -> 504.0 mm, vias 20 -> 19
- net LOPY_CS2: track 93.0 -> 96.0 mm
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Other:
- board text added: "TTL3"
