File: v2.0.brd (EAGLE design)
At the start: 225 x 105 mm, 238 parts, among them J1 DC-044-A, J10 16p-2.54, J11 16p-2.54, J12 4p-2.54, J2 MICROSD-9P, J3 2p-2.54, J4 2p-2.54, J5 16p-2.54, J6 16p-2.54, J7 16p-2.54, J9 16p-2.54, Q10 S8550, Q2 SSM3J328R,LF, Q3 BSS138W-7-F, Q4 BSS138W-7-F, Q5 SSM3J328R,LF, Q6 BSS138W-7-F, Q7 BSS138W-7-F, Q8 CJ2305, Q9 S8550, SW1 MK-12C02 G1.5, SW2 MK-12C02 G1.5, SW3 MK-12C02 G1.5, SW4 MK-12C02 G1.5, U1 MCP23017-E/SO, U10 74HCT139D, U11 BZX84C30, U12 SP483ECN-L, U13 FT232RL-SSOP28, U14 FT232RL-SSOP28, U15 FT232RL-SSOP28, U2 DS3231SN, U3 LOPY, U4 MAX213IDBR, U5 FT232RL-SSOP28, U8 BR24G32-3, Y2 12MHZ

Commit message: As submitted
Parts:
- moved C30 0.76 mm to (13.7, 11.8)
- moved C28 0.51 mm to (13.2, 14.0)
Routing:
- net N$68: track 11.8 -> 9.84 mm
- net USB_HUB_VD33_O: track 12.7 -> 11.9 mm
- net 5V_USB_HUB_FERRITE: track 189.4 -> 190.1 mm
