File: v2.0.sch (EAGLE design)
At the start: 289 parts, among them J1 DC-044-A, J10 16p-2.54, J11 16p-2.54, J2 MICROSD-9P, J3 2p-2.54, J4 2p-2.54, J5 16p-2.54, J6 16p-2.54, J7 16p-2.54, J8 2p-2.54, J9 16p-2.54, Q1 32.768khZ@6Pf, Q10 S8550, Q2 SSM3J328R,LF, Q3 BSS138W-7-F, Q4 BSS138W-7-F, Q5 SSM3J328R,LF, Q6 BSS138W-7-F, Q7 BSS138W-7-F, Q8 CJ2305, Q9 S8550, SW1 MK-12C02 G1.5, SW2 MK-12C02 G1.5, SW3 MK-12C02 G1.5, SW4 MK-12C02 G1.5, U1 MCP23017-E/SO, U10 74HCT139D, U11 BZX84C30, U12 SP483ECN-L, U13 FT232RL-SSOP28, U14 FT232RL-SSOP28, U15 FT232RL-SSOP28, U2 MCP79412-I/SN, U3 LOPY, U4 MAX213IDBR, U5 FT232RL-SSOP28, U6 FT232RL-SSOP28, U8 BR24G32-3, Y2 12MHZ

Commit message: Start of connector / fuse rationalisation
Parts:
- removed C15, C16: 100nf, Seeed-Capacitor-2016:CERAMIC-100NF-50V-10%-X7R(0603)
- removed C17: 4.7uf, Seeed-Capacitor:TANTALUM-SMD-4.7UF-16V(AVX-A)
- removed C9: 10nf, Seeed-Capacitor-2016:CERAMIC-10NF-50V-5%-X7R(0805)
- removed D10: RED-0603, Seeed-LED-2016:LED-SMD-RED-DIFFUSED(0603)
- removed D2: BLUE-0603, Seeed-LED:SMD-LED-CLEAR-BLUE(0603)
- removed D3: GREEN-0603, Seeed-LED:SMD-LED-CLEAR-GREEN(0603)
- removed F11, F12, F13, F14, F17, F18, F2, F21, F22, F23, F24, F25, F3, F30, F31, F32, F33, F34, F35, F36, F37, F38, F39, F4, F44, F45, F52, F53, F7, F8, F80, F81: SMD1206R500SF, Seeed-Fuse:SMD-PPTC-500MA(1206)
- removed I2C_10, I2C_5: JST-XH-05-PIN-ROUND-PAD, Rembrandt Electronics - JST XH Connectors v1-0 2:JST-XH-05-PIN-ROUND-PAD
- removed L1: 330R-1500MA, Seeed-Inductor-2016:SMD-FERRITE-BEAD-330R-1500MA(0805)'0805'
- removed R1, R3: 330R, Seeed-Resistor:SMD-RES-330R-1%-1/10W(0603)
- removed R11: 1K, Seeed-Resistor-2016:SMD-RES-1K-1%-1/10W(0603)
- removed R13, R14: 0R, Seeed-Resistor:SMD-RES-0R-5%-1/10W(0603)
- removed SPI_3, SPI_4, SPI_7, SPI_8: JST-XH-07-PIN-ROUND-PAD, Rembrandt Electronics - JST XH Connectors v1-0 2:JST-XH-07-PIN-ROUND-PAD
- removed TP5: TPB2,54, testpad:TPB2,54
- removed U6: FT232RL-SSOP28, Seeed-IC:INTERFACE-FT232RL(SSOP28)
- removed USB3: ZX62-B-5PA, Seeed-Connector -2016:MICRO-USB-SMD(ZX62-B-5PA)
- added J12: 4p-2.54, Seeed-Connector:DIP-BLACK-FEMALE-HEADER-VERT(4P-2.54)
- added JP1: (no value), jumper:JP1E
Connections:
- removed net ADC_2_3V3_P: F39.2, PI_ADC_2-2.S
- removed net ADC_2_5V_P: F38.2, PI_ADC_2-1.S
- removed net ADC_3_3V3_P: F43.2, PI_ADC_3-2.S
- removed net ADC_4_5V_P: F44.2, PI_ADC_4-1.S
- removed net FTDI1_3V3: C16.2, U6.3V3OUT
- removed net LOPY_UART1_3V3_PROTECTED: F81.2, LOPY_UART1-2.S
- removed net LOPY_UART1_5V_PROTECTED: F80.2, LOPY_UART1-1.S
- removed net LOPY_USB_5V: C15.2, C17.+, L1.2, R1.1, R11.2, R3.1, TP5.TP, U6.VCC, U6.VCCIO
- removed net N$10: R14.1, U6.RXD
- removed net N$2: D3.-, U6.CBUS1
- removed net N$3: D2.-, U6.CBUS0
- removed net N$6: D3.+, R3.2
- removed net N$7: D2.+, R1.2
- removed net N$77: D10.+, R11.1
- removed net N$8: R13.1, U6.TXD
- removed net PI_I2C_3V3_1: F8.2, I2C_2-2.S
- removed net PI_I2C_3V3_10: F37.2, I2C_10-2.S
- removed net PI_I2C_3V3_4: F12.2, I2C_4-2.S
- removed net PI_I2C_3V3_5: F14.2, I2C_5-2.S
- removed net PI_I2C_3V3_7: F18.2, I2C_7-2.S
- removed net PI_I2C_3V3_9: F22.2, I2C_9-2.S
- removed net PI_I2C_5V_P1: F7.2, I2C_2-1.S
- removed net PI_I2C_5V_P3: F11.2, I2C_4-1.S
- removed net PI_I2C_5V_P4: F13.2, I2C_5-1.S
- removed net PI_I2C_5V_P6: F17.2, I2C_7-1.S
- removed net PI_I2C_5V_P8: F21.2, I2C_9-1.S
- removed net PI_I2C_5V_P9: F36.2, I2C_10-1.S
- removed net PI_SPI_5V_2_P: F2.2, SPI_2-1.S
- removed net PI_UART_HUB_2_3V3_P: F53.2, PI_UART_HUB_2-2.S
- removed net PI_UART_HUB_2_5V_P: F52.2, PI_UART_HUB_2-1.S
- removed net RPI_CS8: SPI_8-3.S, U10.2~Y3
- removed net SPI_3V3_2_P: F3.2, SPI_2-2.S
- removed net SPI_3V3_3_P: F23.2, SPI_3-2.S
- removed net SPI_3V3_4_P: F25.2, SPI_4-2.S
- removed net SPI_3V3_6_P: F31.2, SPI_6-2.S
- removed net SPI_3V3_7_P: F33.2, SPI_7-2.S
- removed net SPI_3V3_8_P: F35.2, SPI_8-2.S
- removed net SPI_5V_3_P: F4.2, SPI_3-1.S
- removed net SPI_5V_4_P: F24.2, SPI_4-1.S
- removed net SPI_5V_6_P: F30.2, SPI_6-1.S
- removed net SPI_5V_7_P: F32.2, SPI_7-1.S
- removed net SPI_5V_8_P: F34.2, SPI_8-1.S
- removed net USB_DM: U6.USBDM, USB3.D-
- removed net USB_DP: U6.USBDP, USB3.D+
- removed net VBUS: C9.2, L1.1, USB3.VBUS
- new net RPI_CS0: SPI_1-3.S, U10.1~Y0
- net +3V3: no longer F12.1, F14.1, F18.1, F22.1, F23.1, F25.1, F3.1, F31.1, F33.1, F35.1, F37.1, F53.1, F8.1
- net +3V3_SMOOTH: no longer F39.1, F45.1
- net +5V: now also JP1.1; no longer F80.1
- net ADC_1_3V3_P: now also PI_ADC_2-2.S
- net ADC_1_5V_P: now also PI_ADC_2-1.S
- net ADC_3_5V_P: now also PI_ADC_4-1.S
- net ADC_4_3V3_P: now also F43.2, PI_ADC_3-2.S; no longer F45.2
- net GND: now also JP1.2; no longer C15.1, C16.1, C17.-, C9.1, I2C_10-5.S, I2C_5-5.S, SPI_3-7.S, SPI_4-7.S, SPI_7-7.S, SPI_8-7.S, U6.GND, U6.GND@1, U6.GND@2, U6.GND@A, U6.TEST, USB3.GND, USB3.SHIELD
- net LED_GND: no longer D10.-
- net LOPY_3V3: no longer F81.1
- net LOPY_RXD0: no longer R13.2
- net LOPY_TXD0: no longer R14.2
- net LOPY_UART0_3V3_PROTECTED: now also LOPY_UART1-2.S
- net LOPY_UART0_5V_PROTECTED: now also LOPY_UART1-1.S
- net PI_5V: no longer F11.1, F13.1, F17.1, F2.1, F21.1, F24.1, F30.1, F32.1, F34.1, F36.1, F38.1, F4.1, F44.1, F52.1, F7.1
- net PI_5V_SPI_1_P: now also SPI_2-1.S
- net PI_I2C_3V3_2: now also I2C_4-2.S
- net PI_I2C_3V3_3: now also I2C_2-2.S
- net PI_I2C_3V3_6: now also I2C_7-2.S
- net PI_I2C_3V3_8: now also I2C_9-2.S
- net PI_I2C_5V_P: now also I2C_2-1.S
- net PI_I2C_5V_P2: now also I2C_4-1.S
- net PI_I2C_5V_P5: now also I2C_7-1.S
- net PI_I2C_5V_P7: now also I2C_9-1.S
- net PI_SPI_3V3_1_P: now also SPI_2-2.S
- net PI_UART_HUB_1_3V3_P: now also PI_UART_HUB_2-2.S
- net PI_UART_HUB_1_5V_P: now also PI_UART_HUB_2-1.S
- net RPI_CS1: now also SPI_2-3.S, U10.1~Y1; no longer SPI_1-3.S, U10.1~Y0
- net RPI_CS2: now also SPI_5-3.S, U10.1~Y2; no longer SPI_2-3.S, U10.1~Y1
- net RPI_CS3: now also SPI_6-3.S, U10.1~Y3; no longer SPI_3-3.S, U10.1~Y2
- net RPI_CS4: now also J12.P$1, U10.2~Y0; no longer SPI_4-3.S, U10.1~Y3
- net RPI_CS5: now also J12.P$2, U10.2~Y1; no longer SPI_5-3.S, U10.2~Y0
- net RPI_CS6: now also J12.P$3, U10.2~Y2; no longer SPI_6-3.S, U10.2~Y1
- net RPI_CS7: now also J12.P$4, U10.2~Y3; no longer SPI_7-3.S, U10.2~Y2
- net SCL_3V3: no longer I2C_10-4.S, I2C_5-4.S
- net SDA_3V3: no longer I2C_10-3.S, I2C_5-3.S
- net SPI_3V3_5_P: now also SPI_6-2.S
- net SPI_5V_5_P: now also SPI_6-1.S
- net SPI_MISO: no longer SPI_3-5.S, SPI_4-5.S, SPI_7-5.S, SPI_8-5.S
- net SPI_MOSI: no longer SPI_3-4.S, SPI_4-4.S, SPI_7-4.S, SPI_8-4.S
- net SPI_SCLK: no longer SPI_3-6.S, SPI_4-6.S, SPI_7-6.S, SPI_8-6.S
Other:
- note removed: "Connect for low-level bootloader"
- note removed: "Do we want RST P2 &P12 connected to the Pi because the Pi does weird things to GPIO on boot?"
- note removed: "LoPy FTDI"
- moved on the sheet: F10, F16, F20, F41, F43, F48, F49, F6, LOPY_UART1-1, LOPY_UART1-2, LOPY_UART1-3, LOPY_UART1-4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

Commit message: More rearranging
Parts:
- removed J8: 2p-2.54, Seeed-Connector -2016:DIP-BLACK-ROUND-FEMALE-HEADER-VERT(2P-2.54)
- added F2: SMD1206R500SF, Seeed-Fuse:SMD-PPTC-500MA(1206)
Connections:
- new net N$2: F2.2, JP1.1
- net +5V: now also F2.1; no longer JP1.1
- net EEPROM_WP: no longer J8.1
- net GND: no longer J8.2
Changed lines of the file:
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@@
 <part name="R37" library="Seeed-Resistor-2016" deviceset="SMD-RES-3.9K-5%-1/10W(0603)" device="" value="3.9K"/>
 <part name="R38" library="Seeed-Resistor-2016" deviceset="SMD-RES-3.9K-5%-1/10W(0603)" device="" value="3.9K"/>
-<part name="J8" library="Seeed-Connector -2016" deviceset="DIP-BLACK-ROUND-FEMALE-HEADER-VERT(2P-2.54)" device="" value="2p-2.54"/>
 <part name="TP6" library="testpad" library_urn="urn:adsk.eagle:library:385" deviceset="TP" device="B2,54"/>
 <part name="TP7" library="testpad" library_urn="urn:adsk.eagle:library:385" deviceset="TP" device="B2,54"/>
@@
 <part name="GND26" library="supply1" library_urn="urn:adsk.eagle:library:371" deviceset="GND" device=""/>
 <part name="P+4" library="supply1" library_urn="urn:adsk.eagle:library:371" deviceset="+5V" device=""/>
+<part name="F2" library="Seeed-Fuse" deviceset="SMD-PPTC-500MA(1206)" device="" value="SMD1206R500SF"/>
 </parts>
 <sheets>
@@
 <instance part="R37" gate="G$1" x="365.76" y="176.53" rot="R90"/>
 <instance part="R38" gate="G$1" x="377.19" y="171.45" rot="R90"/>
-<instance part="J8" gate="G$1" x="367.03" y="154.94"/>
 <instance part="TP6" gate="G$1" x="351.79" y="160.02"/>
 <instance part="TP7" gate="G$1" x="355.6" y="154.94"/>
@@
 </segment>
 <segment>
-<pinref part="J8" gate="G$1" pin="2"/>
 <wire x1="359.41" y1="152.4" x2="355.6" y2="152.4" width="0.1524" layer="91"/>
 <pinref part="TP7" gate="G$1" pin="TP"/>
@@
 <wire x1="349.25" y1="177.8" x2="353.06" y2="177.8" width="0.1524" layer="91"/>
 <pinref part="R36" gate="G$1" pin="1"/>
-<pinref part="J8" gate="G$1" pin="1"/>
 <wire x1="359.41" y1="157.48" x2="351.79" y2="157.48" width="0.1524" layer="91"/>
 <wire x1="351.79" y1="157.48" x2="349.25" y2="157.48" width="0.1524" layer="91"/>
@@
 <instance part="JP1" gate="A" x="123.19" y="45.72" rot="R270"/>
 <instance part="GND26" gate="1" x="120.65" y="40.64"/>
-<instance part="P+4" gate="1" x="120.65" y="52.07"/>
+<instance part="P+4" gate="1" x="100.33" y="50.8"/>
+<instance part="F2" gate="G$1" x="111.76" y="45.72"/>
 </instances>
 <busses>
@@
 </segment>
 <segment>
-<pinref part="JP1" gate="A" pin="1"/>
+<pinref part="F2" gate="G$1" pin="1"/>
 <pinref part="P+4" gate="1" pin="+5V"/>
-<wire x1="120.65" y1="45.72" x2="120.65" y2="49.53" width="0.1524" layer="91"/>
+<wire x1="106.68" y1="45.72" x2="100.33" y2="45.72" width="0.1524" layer="91"/>
+<wire x1="100.33" y1="45.72" x2="100.33" y2="48.26" width="0.1524" layer="91"/>
 </segment>
 </net>
@@
 </segment>
 </net>
+<net name="N$2" class="0">
+<segment>
+<pinref part="JP1" gate="A" pin="1"/>
+<pinref part="F2" gate="G$1" pin="2"/>
+<wire x1="120.65" y1="45.72" x2="116.84" y2="45.72" width="0.1524" layer="91"/>
+</segment>
+</net>
